File: Goob/Goob.kicad_sch (KiCad schematic)
At the start: 27 parts, among them J1 Husky Lense, J2 ToF Sensor, J3 SERVO_PAN, J4 SERVO_TILT, J5 SERVO_GATE, J6 MotorA, J7 MotorB, J8 5VIN, SW1 Boot, SW2 EN, U1 ESP32-S3-WROOM-1, U2 Motor Driver, U3 3.3V Reg

Commit message: Initial Commit
Parts:
- added C12: 0.1µF, symbol Device:C
- added C13: 1µF, symbol Device:C
- added F1: 2A hold / ~4A, symbol Device:Polyfuse
- added J9: USB_C_Receptacle_USB2.0_16P, symbol Connector:USB_C_Receptacle_USB2.0_16P
- added Q2, Q3: BSS138, Package_TO_SOT_SMD:SOT-23, symbol Transistor_FET:BSS138
- added R10, R11, R12, R13, R4, R5: 10k, symbol Device:R
- added R6, R7: 5.1k, symbol Device:R
Connections:
- net +3V3: now also J2.1 (Pin_1), C12.1, Q2.1 (G), Q3.1 (G), R10.1, R13.1, R4.1, R5.1
- net +5V: now also F1.2, R11.1, R12.1
- net GND: now also J2.2 (Pin_2), C12.2, C13.2, J9.A1 (GND), J9.A12 (GND), J9.B1 (GND), J9.B12 (GND), J9.SH (SHIELD), R6.2, R7.2
- net I2C_SCL: now also J2.3 (Pin_3), Q2.2 (S), R10.2; no longer J1.4 (Pin_4)
- net I2C_SDA: now also J2.4 (Pin_4), Q3.2 (S), R13.2; no longer J1.3 (Pin_3)
- net TOF_XSHUT: now also J2.6 (Pin_6)
- net IO0: now reaches SW1.1
- net IO0: now also U1.27 (IO0), R4.2
- net EN: now reaches SW2.1
- net EN: now also U1.3 (EN), C13.1, R5.2
- net USB_D−: now reaches U1.13 (USB_D-)
- net USB_D−: now also J9.A7 (D-), J9.B7 (D-)
- net USB_D+: now reaches U1.14 (USB_D+)
- net USB_D+: now also J9.A6 (D+), J9.B6 (D+)
- new net: J9.B5 (CC2), R7.1
- new net: J9.A5 (CC1), R6.1
- new net: F1.1, J9.A4 (VBUS), J9.A9 (VBUS), J9.B4 (VBUS), J9.B9 (VBUS)
- new net HUSKY_SCL_5V: J1.4 (Pin_4), Q2.3 (D), R11.2
- new net HUSKY_SDA_5V: J1.3 (Pin_3), Q3.3 (D), R12.2
- no-connect marks 0 -> 3
Other:
- moved on the sheet: C10, C11, C3, C4, C9, J1, J2, J6, J7, J8, SW1, SW2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
