File: Main/Goob.kicad_sch (KiCad schematic)
At the start: 41 parts, among them J1 Husky Lense, J2 ToF Sensor, J3 SERVO_PAN, J4 SERVO_TILT, J5 SERVO_GATE, J6 MotorA, J7 MotorB, J8 5VIN, J9 USB_C_Receptacle_USB2.0_16P, Q2 BSS138, Q3 BSS138, SW1 Boot, SW2 EN, U1 ESP32-S3-WROOM-1, U2 Motor Driver, U3 3.3V Reg

Commit message: Lots of schematic design
Parts:
- removed J1: Husky Lense, symbol Connector_Generic:Conn_01x04
- removed Q2, Q3: BSS138, Package_TO_SOT_SMD:SOT-23, symbol Transistor_FET:BSS138
- removed R12, R13: 10k, symbol Device:R
- removed SW1: Boot, symbol Switch:SW_Push
- removed SW2: EN, symbol Switch:SW_Push
- added C14: 470µF, Capacitor_THT:CP_Radial_D10.0mm_P5.00mm, symbol Device:C_Polarized
- added C15, C16: 0.1µF, Capacitor_SMD:C_0805_2012Metric, symbol Device:C
- added D1: SS34, Diode_SMD:D_SMA, symbol Diode:SS34
- added J1: Conn_01x03_Pin, Connector_PinHeader_2.54mm:PinHeader_1x03_P2.54mm_Vertical, symbol Connector:Conn_01x03_Pin
- added J10, J12: Conn_01x03, symbol Connector_Generic:Conn_01x03
- added J11: Xiao Connector, Connector_JST:JST_PH_B4B-PH-K_1x04_P2.00mm_Vertical, symbol Connector_Generic:Conn_01x04
- added R8, R9: 4.7k, Resistor_SMD:R_0805_2012Metric, symbol Device:R
- C1, C10, C11, C12, C13, C2, C3, C4, C6, C7, C8, C9: footprint (none) -> Capacitor_SMD:C_0805_2012Metric
- C5: footprint (none) -> Capacitor_THT:CP_Radial_D8.0mm_P3.50mm
- F1: value 2A hold / ~4A -> 2A hold/~4A; footprint (none) -> Fuse:Fuse_1812_4532Metric
- J2: footprint (none) -> Connector_PinHeader_2.54mm:PinHeader_1x06_P2.54mm_Vertical
- J3, J4, J5: footprint (none) -> Connector_PinHeader_2.54mm:PinHeader_1x03_P2.54mm_Vertical
- J6, J7: footprint (none) -> Connector_PinHeader_2.54mm:PinHeader_1x02_P2.54mm_Vertical
- J8: footprint (none) -> TerminalBlock_Phoenix:TerminalBlock_Phoenix_MKDS-1,5-2-5.08_1x02_P5.08mm_Horizontal
- J9: footprint (none) -> Connector_USB:USB_C_Receptacle_GCT_USB4085
- R1, R10, R11, R2, R3, R4, R5, R6, R7: footprint (none) -> Resistor_SMD:R_0805_2012Metric
Connections:
- net HUSKY_SCL_5V is gone; now on net +3V3: R11.2
- net +3V3: now also R10.2, R8.2, R9.2; no longer R10.1
- net +5V: now also C14.1, C15.1, C16.1, D1.1 (K), J10.1 (Pin_1), J11.1 (Pin_1), J12.1 (Pin_1); no longer F1.2, R11.1
- net EN: now also J1.1 (Pin_1)
- net GND: now also C14.2, C15.2, C16.2, J1.3 (Pin_3), J10.2 (Pin_2), J11.2 (Pin_2), J12.2 (Pin_2)
- net I2C_SCL: now also R8.1; no longer R10.2
- net I2C_SDA: now also R9.1
- net IO0: now also J1.2 (Pin_2)
- net VISION_RX: now reaches U1.19 (IO11)
- net VISION_RX: now also J11.4 (Pin_4)
- net VISION_TX: now reaches U1.20 (IO12)
- net VISION_TX: now also J11.3 (Pin_3)
- net FLY_A_TACH: now reaches U1.21 (IO13)
- net FLY_A_TACH: now also R10.1, J10.3 (Pin_3)
- net FLY_B_TACH: now reaches U1.22 (IO14)
- net FLY_B_TACH: now also R11.1, J12.3 (Pin_3)
- new net: D1.2 (A), F1.2
- no-connect marks 3 -> 20
Other:
- moved on the sheet: C11, C12, C13, J2, R4, R5
