File: Main/Main.kicad_sch (KiCad schematic)
At the start: 44 parts, among them J1 Conn_01x03_Pin, J10 Conn_01x03, J11 Xiao Connector, J12 Conn_01x03, J2 ToF Sensor, J3 SERVO_PAN, J4 SERVO_TILT, J5 SERVO_GATE, J6 MotorA, J7 MotorB, J8 5VIN, J9 USB_C_Receptacle_USB2.0_16P, U1 ESP32-S3-WROOM-1, U2 Motor Driver, U3 3.3V Reg

Commit message: Voltage Reg and EN and Boot
Parts:
- renumbered C14 to C16
Other:
- moved on the sheet: C10, C9, U3
