File: Battery/Battery.kicad_pcb (KiCad board)
At the start: 2 copper layers, 3 parts, among them J1 Conn_01x03_Pin, J2 Conn_01x05, J4 Conn_01x04

Commit message: Battery PCB
Parts:
- added J3: Conn_01x02, Connector_JST:JST_PH_B2B-PH-K_1x02_P2.00mm_Vertical, F.Cu at (24.0, 36.5)
- added J5: Conn_01x02, TerminalBlock_Phoenix:TerminalBlock_Phoenix_MKDS-1,5-2-5.08_1x02_P5.08mm_Horizontal, F.Cu at (27.6, 17.5)
- added REF**: MountingHole_3.2mm_M3, MountingHole:MountingHole_3.2mm_M3, F.Cu at (15.5, 15.5)
- added REF**: MountingHole_3.2mm_M3, MountingHole:MountingHole_3.2mm_M3, F.Cu at (15.5, 38.5)
- added REF**: MountingHole_3.2mm_M3, MountingHole:MountingHole_3.2mm_M3, F.Cu at (38.5, 15.5)
- added REF**: MountingHole_3.2mm_M3, MountingHole:MountingHole_3.2mm_M3, F.Cu at (38.5, 38.5)
- added SW1: SW_SPST, Connector_PinHeader_2.54mm:PinHeader_1x02_P2.54mm_Vertical, F.Cu at (33.0, 14.5)
- moved J1 27.5 mm to (15.5, 31.5), turned to 90 degrees
- moved J4 7.59 mm to (40.0, 30.6), turned to 180 degrees
- moved J2 5.23 mm to (35.0, 33.2), turned to 180 degrees
Routing:
- net +5V: track 0.00 -> 35.7 mm, vias 0 -> 1
- net VBATT: track 0.00 -> 29.6 mm, vias 0 -> 1
- net PACK_TOP: track 0.00 -> 20.2 mm
- net PACK_MID: track 0.00 -> 20.2 mm
- net VBATT_SW: track 0.00 -> 16.5 mm, vias 0 -> 1
- added copper zone on B.Cu, net GND
- added copper zone on F.Cu, net GND
Other:
- board outline added: 30 x 30 mm

Commit message: Update net assignments and main board power
Parts:
- moved J2 3.00 mm to (32.5, 31.5)
- moved J3 1.63 mm to (23.5, 38.0)
Routing:
- net VBATT: track 29.6 -> 33.1 mm
- net PACK_TOP: track 20.2 -> 17.0 mm, vias 0 -> 1
- net PACK_MID: track 20.2 -> 17.0 mm, vias 0 -> 1
- net +5V: track 35.7 -> 35.0 mm, vias 1 -> 0
Changed lines of the file:
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@@
 	(footprint "Connector_JST:JST_PH_B2B-PH-K_1x02_P2.00mm_Vertical"
 		(layer "F.Cu")
-		(at 24 36.45)
+		(at 23.5 38)
 		(descr "JST PH series connector, B2B-PH-K (http://www.jst-mfg.com/product/pdf/eng/ePH.pdf)")
 		(tags "connector JST PH vertical")
@@
 	(footprint "Connector_PinHeader_2.54mm:PinHeader_1x05_P2.54mm_Vertical"
 		(layer "F.Cu")
-		(at 35 33.16 180)
+		(at 32.5 31.5 180)
 		(descr "Through hole straight pin header, 1x05, 2.54mm pitch, single row")
 		(tags "Through hole pin header THT 1x05 2.54mm single row")
@@
 	)
 	(segment
-		(start 15.5 31.5)
-		(end 33.34 31.5)
-		(width 0.25)
-		(layer "F.Cu")
-		(net "PACK_TOP")
-	)
-	(segment
-		(start 33.34 31.5)
-		(end 35 33.16)
-		(width 0.25)
-		(layer "F.Cu")
-		(net "PACK_TOP")
-	)
-	(segment
-		(start 33.38 29)
-		(end 35 30.62)
-		(width 0.25)
-		(layer "F.Cu")
-		(net "PACK_MID")
-	)
-	(segment
-		(start 15.5 29)
-		(end 33.38 29)
-		(width 0.25)
-		(layer "F.Cu")
-		(net "PACK_MID")
-	)
-	(segment
-		(start 36.45 17.95)
+		(start 34.85 33.85)
+		(end 33.7 35)
+		(width 2.5)
+		(layer "F.Cu")
+		(net "+5V")
+	)
+	(segment
+		(start 27.58 32.58)
+		(end 27.58 17.5)
+		(width 2.5)
+		(layer "F.Cu")
+		(net "+5V")
+	)
+	(segment
+		(start 33.7 35)
+		(end 30 35)
+		(width 2.5)
+		(layer "F.Cu")
+		(net "+5V")
+	)
+	(segment
+		(start 38.797919 25.54)
+		(end 34.85 29.487919)
+		(width 2.5)
+		(layer "F.Cu")
+		(net "+5V")
+	)
+	(segment
+		(start 40 25.54)
+		(end 38.797919 25.54)
+		(width 2.5)
+		(layer "F.Cu")
+		(net "+5V")
+	)
+	(segment
+		(start 30 35)
+		(end 27.58 32.58)
+		(width 2.5)
+		(layer "F.Cu")
+		(net "+5V")
+	)
+	(segment
+		(start 34.85 29.487919)
+		(end 34.85 33.85)
+		(width 2.5)
+		(layer "F.Cu")
+		(net "+5V")
+	)
+	(segment
+		(start 32.5 23.5)
+		(end 35 21)
+		(width 0.3)
+		(layer "F.Cu")
+		(net "VBATT")
+	)
+	(segment
+		(start 35 21)
+		(end 35 17)
+		(width 0.3)
+		(layer "F.Cu")
+		(net "VBATT")
+	)
+	(segment
+		(start 35 17)
+		(end 33 15)
+		(width 0.3)
+		(layer "F.Cu")
+		(net "VBATT")
+	)
+	(segment
+		(start 33 15)
 		(end 33 14.5)
-		(width 0.8)
+		(width 0.3)
 		(layer "F.Cu")
 		(net "VBATT")
 	)
 	(segment
-		(start 30 32.325)
-		(end 28.125 32.325)
-		(width 0.8)
+		(start 23.5 26)
+		(end 25.5 24)
+		(width 0.3)
 		(layer "F.Cu")
 		(net "VBATT")
 	)
 	(segment
-		(start 36.45 24.09)
-		(end 36.45 17.95)
-		(width 0.8)
+		(start 23.5 38)
+		(end 23.5 26)
+		(width 0.3)
 		(layer "F.Cu")
 		(net "VBATT")
 	)
 	(segment
-		(start 35 25.54)
-		(end 36.45 24.09)
-		(width 0.8)
+		(start 32.5 23.88)
+		(end 32.5 23.5)
+		(width 0.3)
 		(layer "F.Cu")
 		(net "VBATT")
 	)
-	(segment
-		(start 28.125 32.325)
-		(end 24 36.45)
-		(width 0.8)
-		(layer "F.Cu")
-		(net "VBATT")
-	)
 	(via
-		(at 30 32.325)
-		(size 1)
-		(drill 0.5)
+		(at 25.5 24)
+		(size 0.6)
+		(drill 0.3)
 		(layers "F.Cu" "B.Cu")
 		(net "VBATT")
 	)
 	(segment
-		(start 32.5 29.825)
-		(end 32.5 28.04)
-		(width 0.8)
+		(start 25.5 24)
+		(end 25.62 23.88)
+		(width 0.3)
 		(layer "B.Cu")
 		(net "VBATT")
 	)
 	(segment
-		(start 30 32.325)
-		(end 32.5 29.825)
-		(width 0.8)
+		(start 25.62 23.88)
+		(end 32.5 23.88)
+		(width 0.3)
 		(layer "B.Cu")
 		(net "VBATT")
 	)
 	(segment
-		(start 32.5 28.04)
-		(end 35 25.54)
-		(width 0.8)
-		(layer "B.Cu")
-		(net "VBATT")
-	)
-	(segment
 		(start 33 17.04)
 		(end 33 18.5)
-		(width 0.8)
+		(width 0.3)
 		(layer "F.Cu")
 		(net "VBATT_SW")
@@
 	(segment
 		(start 33 18.5)
-		(end 35 20.5)
-		(width 0.8)
+		(end 34 19.5)
+		(width 0.3)
 		(layer "F.Cu")
 		(net "VBATT_SW")
 	)
 	(via
-		(at 35 20.5)
-		(size 1)
-		(drill 0.5)
+		(at 34 19.5)
+		(size 0.6)
+		(drill 0.3)
 		(layers "F.Cu" "B.Cu")
 		(net "VBATT_SW")
 	)
 	(segment
-		(start 35 20.5)
-		(end 38.55 24.05)
-		(width 0.8)
+		(start 34 19.5)
+		(end 38.75 24.25)
+		(width 0.3)
 		(layer "B.Cu")
 		(net "VBATT_SW")
 	)
 	(segment
-		(start 38.55 24.05)
-		(end 38.55 29.17)
-		(width 0.8)
+		(start 38.75 29.37)
+		(end 40 30.62)
+		(width 0.3)
 		(layer "B.Cu")
 		(net "VBATT_SW")
 	)
 	(segment
-		(start 38.55 29.17)
-		(end 40 30.62)
-		(width 0.8)
+		(start 38.75 24.25)
+		(end 38.75 29.37)
+		(width 0.3)
 		(layer "B.Cu")
 		(net "VBATT_SW")
 	)
 	(segment
-		(start 36.39 34.61)
-		(end 36.45 34.61)
-		(width 0.8)
-		(layer "F.Cu")
-		(net "+5V")
-	)
-	(segment
-		(start 36.45 29.09)
-		(end 40 25.54)
-		(width 0.8)
-		(layer "F.Cu")
-		(net "+5V")
-	)
-	(segment
-		(start 36.45 34.61)
-		(end 36.45 29.09)
-		(width 0.8)
-		(layer "F.Cu")
-		(net "+5V")
-	)
-	(segment
-		(start 35.5 35.5)
-		(end 36.39 34.61)
-		(width 0.8)
-		(layer "F.Cu")
-		(net "+5V")
-	)
-	(segment
-		(start 31.175 35.5)
-		(end 35.5 35.5)
-		(width 0.8)
-		(layer "F.Cu")
-		(net "+5V")
-	)
-	(segment
-		(start 29.5875 33.9125)
-		(end 31.175 35.5)
-		(width 0.8)
-		(layer "F.Cu")
-		(net "+5V")
+		(start 15.5 31.5)
+		(end 22.5 31.5)
+		(width 0.3)
+		(layer "F.Cu")
+		(net "PACK_TOP")
 	)
 	(via
-		(at 29.5875 33.9125)
-		(size 1)
-		(drill 0.5)
+		(at 22.5 31.5)
+		(size 0.6)
+		(drill 0.3)
 		(layers "F.Cu" "B.Cu")
-		(net "+5V")
-	)
-	(segment
-		(start 27.58 31.905)
-		(end 27.58 17.5)
-		(width 0.8)
+		(net "PACK_TOP")
+	)
+	(segment
+		(start 22.5 31.5)
+		(end 32.5 31.5)
+		(width 0.3)
 		(layer "B.Cu")
-		(net "+5V")
-	)
-	(segment
-		(start 29.5875 33.9125)
-		(end 27.58 31.905)
-		(width 0.8)
+		(net "PACK_TOP")
+	)
+	(segment
+		(start 15.5 29)
+		(end 22.5 29)
+		(width 0.3)
+		(layer "F.Cu")
+		(net "PACK_MID")
+	)
+	(via
+		(at 22.5 29)
+		(size 0.6)
+		(drill 0.3)
+		(layers "F.Cu" "B.Cu")
+		(net "PACK_MID")
+	)
+	(segment
+		(start 25.82 28.96)
+		(end 32.5 28.96)
+		(width 0.3)
 		(layer "B.Cu")
-		(net "+5V")
+		(net "PACK_MID")
+	)
+	(segment
+		(start 22.5 29)
+		(end 25.78 29)
+		(width 0.3)
+		(layer "B.Cu")
+		(net "PACK_MID")
+	)
+	(segment
+		(start 25.78 29)
+		(end 25.82 28.96)
+		(width 0.3)
+		(layer "B.Cu")
+		(net "PACK_MID")
 	)
 	(zone
